File: PCB/openDTU.kicad_pcb (KiCad board)
At the start: 2 copper layers, 60 x 50 mm, 18 parts, among them U1 ESP32NodeMCU, U2 NRF24L01+PA+LNA_Breakout

Commit message: Updated to REV2.1
Parts:
- removed the REF** at (117.7, 72.9)
- removed the REF** at (172.7, 72.9)
- removed the REF** at (172.7, 117.9)
- removed the REF** at (117.7, 117.9)
- moved G*** 42.4 mm to (168.2, 73.4)
- moved C1 11.1 mm to (162.1, 113.4), turned to 90 degrees
- moved REF** 6.67 mm to (160.7, 80.9)
- moved G*** 3.52 mm to (154.2, 118.9)
- moved U2 3.12 mm to (158.1, 107.0)
Routing:
- net +3.3V: track 83.7 -> 124.0 mm
- net /IRQ: track 33.1 -> 30.0 mm
- net /CE: track 26.5 -> 23.9 mm
- net /MOSI: track 51.9 -> 49.9 mm
- net /MISO: track 40.4 -> 39.3 mm
- net /SCK: track 35.8 -> 34.8 mm
- net /~{CSN}: track 29.7 -> 29.0 mm
- net GND: vias 26 -> 30
Other:
- board size 60 x 50 mm -> 60 x 55 mm
- board text added: "REV2.1 2023/02"
- board text removed: "REV2.0 2023/01"
