File: openDTU.kicad_pcb (KiCad board)
At the start: 2 copper layers, 60 x 55 mm, 14 parts, among them U1 ESP32NodeMCU, U2 NRF24L01+PA+LNA_Breakout

Commit message: Updated Board to REV2.1
Other:
- board text added: "REV2.2 2023/02"
Changed lines of the file:
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@@
   (title_block
     (title "openDTU-BreakoutBoard")
-    (date "2023-02-18")
-    (rev "2.1")
+    (date "2023-02-25")
+    (rev "2.2")
   )
   (layers
@@
     (pad_to_mask_clearance 0)
     (aux_axis_origin 115.18 70.396)
-    (grid_origin 115.18 70.396)
+    (grid_origin 154.36 80.166)
     (pcbplotparams
       (layerselection 0x00010fc_ffffffff)
@@
     (pad "38" thru_hole rect (at 25.4 0) (size 1.7 1.7) (drill 1) (layers "*.Cu" "*.Mask")
       (net 14 "GND") (pinfunction "GND") (pintype "passive"))
-    (model "${KICAD6_3DMODEL_DIR}/Connector_PinSocket_2.54mm.3dshapes/PinSocket_1x19_P2.54mm_Vertical.wrl"
-      (offset (xyz 0 0 0))
-      (scale (xyz 1 1 1))
-      (rotate (xyz 0 0 0))
-    )
-    (model "${KICAD6_3DMODEL_DIR}/Connector_PinSocket_2.54mm.3dshapes/PinSocket_1x19_P2.54mm_Vertical.wrl"
-      (offset (xyz 25.4 0 0))
-      (scale (xyz 1 1 1))
-      (rotate (xyz 0 0 0))
-    )
     (model "${KIPRJMOD}/Libraries/ESP32-NodeMCU_WROOM_32/ESP32-NodeMCU_WROOM_32.STEP"
-      (offset (xyz 12.7 -22.86 10.16))
+      (offset (xyz 12.7 -22.86 2.64))
       (scale (xyz 1 1 1))
       (rotate (xyz -90 0 0))
@@
       (net 27 "/IRQ") (pinfunction "IRQ") (pintype "output"))
     (model "${KIPRJMOD}/Libraries/nRF24L01+PA+LNA/NRF24L01+PA+LNA.STEP"
-      (offset (xyz -1.905 -3.81 9.65))
+      (offset (xyz -1.905 -3.81 2.64))
       (scale (xyz 1 1 1))
       (rotate (xyz -90 0 0))
     )
-    (model "${KICAD6_3DMODEL_DIR}/Connector_PinSocket_2.54mm.3dshapes/PinSocket_2x04_P2.54mm_Vertical.wrl"
-      (offset (xyz 2.5 0 0))
-      (scale (xyz 1 1 1))
-      (rotate (xyz 0 0 0))
-    )
   )
   (footprint "TestPoint:TestPoint_THTPad_D1.5mm_Drill0.7mm" (layer "F.Cu")
@@
     (effects (font (size 1.5 2) (thickness 0.25)) (justify left mirror))
   )
-  (gr_text "REV2.1 2023/02" (at 157.87417 120.4446) (layer "F.SilkS")
+  (gr_text "REV2.2 2023/02" (at 157.87417 120.4446) (layer "F.SilkS")
     (effects (font (size 1 1) (thickness 0.15)) (justify left))
   )
@@
       )
     )
+  )
+  (zone (net 0) (net_name "") (layers "F&B.Cu") (name "ESP32 WiFi ") (hatch full 0.508)
+    (connect_pads (clearance 0))
+    (min_thickness 0.254) (filled_areas_thickness no)
+    (keepout (tracks allowed) (vias allowed) (pads allowed) (copperpour not_allowed) (footprints allowed))
+    (fill (thermal_gap 0.508) (thermal_bridge_width 0.508))
+    (polygon
+      (pts
+        (xy 167.86 77.666)
+        (xy 167.36 78.166)
+        (xy 166.86 78.666)
+        (xy 161.86 78.666)
+        (xy 156.86 78.666)
+        (xy 156.36 78.166)
+        (xy 155.86 77.666)
+        (xy 155.86 75.721)
+        (xy 155.86 67.916)
+        (xy 167.86 67.916)
+      )
+    )
